Commit message: feat: 증속벨트반영, drive 인자로 구동 구성 선택

File: workspace/ros2_ws/src/opencr_hardware/urdf/opencr.ros2_control.xacro (robot description, xacro)
@@ -29,5 +29,5 @@
   <!-- 두 OpenCR의 순서는 고정하지 않고 STATE.role로 역할을 판별한다. -->
   <!-- wheel_count 4 의 칸 순서 (왼앞 0 · 왼뒤 1 · 오른앞 2 · 오른뒤 3) 는 주행 펌웨어 config.h WHEEL_IDS · WHEEL_DIR 와 같다 -->
-  <xacro:macro name="opencr_ros2_control" params="name:=OpenCRSystem ports:=/dev/ttyACM0,/dev/ttyACM1 wheel_count:=4 use_gripper:=false joy_required:=true">
+  <xacro:macro name="opencr_ros2_control" params="name:=OpenCRSystem ports:=/dev/ttyACM0,/dev/ttyACM1 wheel_count:=4 use_gripper:=false joy_required:=true wheel_gear:=1.0">
     <ros2_control name="${name}" type="system">
       <hardware>
@@ -43,4 +43,6 @@
         <param name="battery_warn_v">11.1</param>
         <param name="battery_error_v">10.5</param>
+        <!-- 바퀴 각속도 / 모터 각속도. 펌웨어는 모터 축 기준 (WHEEL_GEAR 1.0 고정), 변환은 하드웨어 인터페이스가 한다 -->
+        <param name="wheel_gear">${wheel_gear}</param>
       </hardware>
       <xacro:if value="${wheel_count == 4}">

File: workspace/ros2_ws/src/opencr_hardware/urdf/robot.urdf.xacro (robot description, xacro)
@@ -8,11 +8,21 @@
   <xacro:arg name="ports" default="/dev/ttyACM0,/dev/ttyACM1"/>
   <xacro:arg name="joy_required" default="true"/>
+  <!-- 구동 방식: belt = 증속벨트 1:1.5 (2026-10-27 장착), direct = 직결 (urdfv2). 바퀴 y · 한계 · 기어비가 같이 바뀐다 -->
+  <xacro:arg name="drive" default="belt"/>
   <xacro:include filename="$(find opencr_hardware)/urdf/opencr.ros2_control.xacro"/>
   <xacro:property name="wheel_count" value="$(arg wheel_count)"/>
+  <xacro:property name="drive" value="$(arg drive)"/>
+  <xacro:if value="${drive not in ['direct', 'belt']}">
+    ${xacro.fatal("drive 는 direct 또는 belt: " + drive)}
+  </xacro:if>
+  <xacro:property name="belt" value="${drive == 'belt'}"/>
   <!-- 바퀴 · 차체 높이 · IMU 는 기준 URDF urdfv2/urdf/teamrobot.urdf (teamrobot_4wd, 직결) 값 (2026-10-26).
        base_link 원점 = urdfv2 와 같음 (하판 윗면 중심, 바닥 위 56.25 mm). 관절 이름은 ros2_control · 컨트롤러 설정 때문에 기존 이름 유지:
        wheel_left_front = wheel_fl · wheel_left_rear = wheel_rl · wheel_right_front = wheel_fr · wheel_right_rear = wheel_rr -->
-  <xacro:property name="wheel_y" value="0.1372"/>     <!-- 바퀴 중심 |y| (직결, 바퀴 간격 0.2744) -->
-  <xacro:property name="wheel_x" value="0.100"/>      <!-- 앞바퀴 x, 뒤바퀴 x = -0.100 (앞뒤 대칭) -->
+  <!-- belt: 증속벨트 설계 (구동_증속벨트 drive_belt.scad · ref/wheels_shifted15.stl) — 바퀴를 바깥으로 15 mm, x · 축 높이는 직결과 같음.
+       y 0.1585 는 설계 차체 기준 절대값 (설계 직결 |y| 143.5 ≠ urdfv2 직결 137.2) ★ 장착 후 바퀴 간격 실측 -->
+  <xacro:property name="wheel_y" value="${0.1585 if belt else 0.1372}"/>   <!-- 바퀴 중심 |y| (간격 belt 0.317 · direct 0.2744) -->
+  <xacro:property name="wheel_x" value="0.100"/>      <!-- 앞바퀴 x, 뒤바퀴 x = -0.100 (앞뒤 대칭, belt · direct 같음) -->
+  <xacro:property name="wheel_gear" value="${1.5 if belt else 1.0}"/>      <!-- 바퀴 각속도 / 모터 각속도 (모터 36T → 바퀴 24T) -->
   <xacro:property name="wheel_z" value="-0.02325"/>   <!-- 바퀴 중심 z (base_link 아래) -->
   <xacro:property name="wheel_radius" value="0.033"/> <!-- Ø66. controllers_4wd.yaml wheel_radius 와 같게 -->
@@ -33,5 +43,6 @@
       <origin xyz="${x} ${y} ${wheel_z}" rpy="0 0 0"/>
       <axis xyz="0 1 0"/>
-      <limit effort="3.0" velocity="8.063421"/>   <!-- XM430-W210 12 V: 3.0 N·m, 무부하 77 rpm (직결) -->
+      <!-- XM430-W210 12 V: 3.0 N·m, 무부하 77 rpm (8.063 rad/s) → 바퀴 기준 토크 ÷ 기어비, 속도 × 기어비 -->
+      <limit effort="${3.0 / wheel_gear}" velocity="${8.063421 * wheel_gear}"/>
     </joint>
   </xacro:macro>
@@ -82,4 +93,4 @@
   <xacro:fixed_link name="tool_link"       parent="gripper_roll_link" xyz="0.086 0 0" rpy="0 0 0"/>
   <xacro:opencr_ros2_control ports="$(arg ports)" wheel_count="${wheel_count}" use_gripper="$(arg use_gripper)"
-                             joy_required="$(arg joy_required)"/>
+                             joy_required="$(arg joy_required)" wheel_gear="${wheel_gear}"/>
 </robot>

Commit message: feat: Isaac Sim 6.2 브리지 추가, TopicBasedSystem 연결

File: workspace/ros2_ws/src/opencr_hardware/urdf/opencr.ros2_control.xacro (robot description, xacro)
@@ -29,7 +29,14 @@
   <!-- 두 OpenCR의 순서는 고정하지 않고 STATE.role로 역할을 판별한다. -->
   <!-- wheel_count 4 의 칸 순서 (왼앞 0 · 왼뒤 1 · 오른앞 2 · 오른뒤 3) 는 주행 펌웨어 config.h WHEEL_IDS · WHEEL_DIR 와 같다 -->
-  <xacro:macro name="opencr_ros2_control" params="name:=OpenCRSystem ports:=/dev/ttyACM0,/dev/ttyACM1 wheel_count:=4 use_gripper:=false joy_required:=true wheel_gear:=1.0">
+  <!-- sim: Isaac Sim — OpenCRHardware 대신 TopicBasedSystem 이 관절 상태 · 명령을 토픽으로 주고받는다 (브리지 workspace/tools/isaac_sim) -->
+  <xacro:macro name="opencr_ros2_control" params="name:=OpenCRSystem ports:=/dev/ttyACM0,/dev/ttyACM1 wheel_count:=4 use_gripper:=false joy_required:=true wheel_gear:=1.0 sim:=false">
     <ros2_control name="${name}" type="system">
       <hardware>
+        <xacro:if value="${sim}">
+        <plugin>topic_based_ros2_control/TopicBasedSystem</plugin>
+        <param name="joint_commands_topic">/isaac_joint_commands</param>
+        <param name="joint_states_topic">/isaac_joint_states</param>
+        </xacro:if>
+        <xacro:unless value="${sim}">
         <plugin>opencr_hardware/OpenCRHardware</plugin>
         <param name="ports">${ports}</param>
@@ -45,4 +52,5 @@
         <!-- 바퀴 각속도 / 모터 각속도. 펌웨어는 모터 축 기준 (WHEEL_GEAR 1.0 고정), 변환은 하드웨어 인터페이스가 한다 -->
         <param name="wheel_gear">${wheel_gear}</param>
+        </xacro:unless>
       </hardware>
       <xacro:if value="${wheel_count == 4}">
@@ -78,4 +86,6 @@
         </joint>
       </xacro:if>
+      <!-- TopicBasedSystem 은 센서를 다루지 않는다 — 시뮬레이션은 브리지가 /imu/data 를 직접 발행 -->
+      <xacro:unless value="${sim}">
       <sensor name="imu">
         <state_interface name="orientation.x"/>
@@ -90,4 +100,5 @@
         <state_interface name="linear_acceleration.z"/>
       </sensor>
+      </xacro:unless>
     </ros2_control>
   </xacro:macro>

File: workspace/ros2_ws/src/opencr_hardware/urdf/robot.urdf.xacro (robot description, xacro)
@@ -10,4 +10,5 @@
   <!-- 구동 방식: belt = 증속벨트 1:1.5 (2026-10-27 장착), direct = 직결 (urdfv2). 바퀴 y · 한계 · 기어비가 같이 바뀐다 -->
   <xacro:arg name="drive" default="belt"/>
+  <xacro:arg name="sim" default="false"/>   <!-- Isaac Sim: TopicBasedSystem (opencr.ros2_control.xacro) -->
   <xacro:include filename="$(find opencr_hardware)/urdf/opencr.ros2_control.xacro"/>
   <xacro:property name="wheel_count" value="$(arg wheel_count)"/>
@@ -104,4 +105,4 @@
   <xacro:fixed_link name="tool_link"       parent="gripper_roll_link" xyz="0.086 0 0" rpy="0 0 0"/>
   <xacro:opencr_ros2_control ports="$(arg ports)" wheel_count="${wheel_count}" use_gripper="$(arg use_gripper)"
-                             joy_required="$(arg joy_required)" wheel_gear="${wheel_gear}"/>
+                             joy_required="$(arg joy_required)" wheel_gear="${wheel_gear}" sim="$(arg sim)"/>
 </robot>
